File: Kicad/MX_HHKB.kicad_pcb (KiCad board)
At the start: 2 copper layers, 285.1 x 94.3 mm, 171 parts, among them J1 USB_mini_micro_B, K1 K00, K10 K09, K11 K0A, K12 K0B, K13 K0C, K14 K10, K15 K11, K16 K12, K17 K13, K18 K14, K19 K15, K2 K01, K20 K16, K21 K17, K22 K18, K23 K19, K24 K1A, K25 K1B, K26 K1C, K27 K20, K28 K21, K29 K22, K3 K02, K30 K23, K31 K24, K32 K25, K33 K26, K34 K27, K35 K28, K36 K29, K37 K2A, K38 K2B, K39 K2C, K4 K03, K40 K30, K41 K31, K42 K32, K43 K33, K44 K34, K45 K35, K46 K36, K47 K37, K48 K38, K49 K39, K5 K04, K50 K3A, K51 K3B, K52 K3C, K53 K41, K54 K42, K55 K45, K56 K48, K57 K49, K58 K4A, K59 K4B, K6 K05, K60 K4C, K61 Ctrl, K62 L_ALT, K63 SPACE, K64 SPACE, K65 R_ALT, K66 R_ALT, K67 R_GUI, K68 R_GUI, K69 K30, K7 K06, K70 K3C, K71 K3B, K72 SPACE, K8 K07, K9 K08, SW1 SW_PUSH, U0 ATMEGA32U4, X1 XTAL_GND

Commit message: - Moved d25
Parts:
- moved D32 5.94 mm to (185.0, 150.0), turned to 0 degrees
Routing:
- net /Row2: track 475.6 -> 480.0 mm
Changed lines of the file:
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@@
     (thickness 1.6)
     (drawings 26)
-    (tracks 1111)
+    (tracks 1113)
     (zones 0)
     (modules 171)
@@
   )
   (module Footprint:D_SOD123 (layer B.Cu)
-    (at 190.75 151.5 90)
+    (at 185 150)
     (attr smd)
-    (fp_text reference D32 (at 0 -1.925 90) (layer B.SilkS) hide
+    (fp_text reference D32 (at 0 -1.925) (layer B.SilkS) hide
       (effects (font (size 0.8 0.8) (thickness 0.15)) (justify mirror))
     )
-    (fp_text value D25 (at 0 1.925 90) (layer B.SilkS)
+    (fp_text value D25 (at 0 1.925) (layer B.SilkS) hide
       (effects (font (size 0.8 0.8) (thickness 0.15)) (justify mirror))
     )
@@
     (fp_line (start 2.8 -1.2) (end -3.2 -1.2) (layer B.SilkS) (width 0.2))
     (fp_line (start -3.2 -1.2) (end -3.2 1.2) (layer B.SilkS) (width 0.2))
-    (pad 2 smd rect (at 1.7 0 90) (size 1.2 1.4) (layers B.Cu B.Paste B.Mask)
+    (pad 2 smd rect (at 1.7 0) (size 1.2 1.4) (layers B.Cu B.Paste B.Mask)
       (net 40 "Net-(D32-Pad2)"))
-    (pad 1 smd rect (at -1.7 0 90) (size 1.2 1.4) (layers B.Cu B.Paste B.Mask)
+    (pad 1 smd rect (at -1.7 0) (size 1.2 1.4) (layers B.Cu B.Paste B.Mask)
       (net 35 /Row2))
   )
@@
   (segment (start 83.75 138) (end 79.1625 138) (width 0.25) (layer B.Cu) (net 34))
   (segment (start 75.175 141.9875) (end 75.17625 141.98625) (width 0.25) (layer B.Cu) (net 34))
+  (segment (start 209.65 154) (end 207.049998 156.600002) (width 0.25) (layer B.Cu) (net 35))
+  (segment (start 207.049998 156.600002) (end 207.049998 158) (width 0.25) (layer B.Cu) (net 35))
+  (segment (start 183.3 150) (end 183.3 150.05) (width 0.25) (layer B.Cu) (net 35) (status C00000))
+  (segment (start 183.3 150.05) (end 187.25 154) (width 0.25) (layer B.Cu) (net 35) (status 400000))
+  (segment (start 209.65 154) (end 214.3125 149.3375) (width 0.25) (layer B.Cu) (net 35) (status 800000))
+  (segment (start 187.25 154) (end 209.65 154) (width 0.25) (layer B.Cu) (net 35))
+  (segment (start 176.2125 149.3375) (end 182.6375 149.3375) (width 0.25) (layer B.Cu) (net 35) (status 400000))
+  (segment (start 182.6375 149.3375) (end 183.3 150) (width 0.25) (layer B.Cu) (net 35) (status 800000))
+  (segment (start 210.4 153.25) (end 214.3125 149.3375) (width 0.25) (layer B.Cu) (net 35))
   (segment (start 339.75 147.45) (end 333.3 147.45) (width 0.25) (layer B.Cu) (net 35))
   (segment (start 333.3 147.45) (end 331.4125 149.3375) (width 0.25) (layer B.Cu) (net 35))
-  (segment (start 176.2125 149.3375) (end 186.8875 149.3375) (width 0.25) (layer B.Cu) (net 35))
-  (segment (start 186.8875 149.3375) (end 190.75 153.2) (width 0.25) (layer B.Cu) (net 35))
-  (segment (start 194.5 153.25) (end 190.8 153.25) (width 0.25) (layer B.Cu) (net 35))
-  (segment (start 190.8 153.25) (end 190.75 153.2) (width 0.25) (layer B.Cu) (net 35))
-  (segment (start 207.049998 160.75) (end 207.049998 157.799998) (width 0.25) (layer B.Cu) (net 35))
-  (segment (start 207.049998 157.799998) (end 202.5 153.25) (width 0.25) (layer B.Cu) (net 35))
+  (segment (start 207.049998 160.75) (end 207.049998 158) (width 0.25) (layer B.Cu) (net 35))
+  (segment (start 207.049998 158) (end 207.049998 157.799998) (width 0.25) (layer B.Cu) (net 35))
   (segment (start 143.5 187.75) (end 220.5 187.75) (width 0.25) (layer B.Cu) (net 35))
   (segment (start 220.5 187.75) (end 222.5 185.75) (width 0.25) (layer B.Cu) (net 35))
@@
   (segment (start 111.011396 191.350002) (end 78.463604 191.350002) (width 0.25) (layer B.Cu) (net 35))
   (segment (start 112.805699 189.555699) (end 111.011396 191.350002) (width 0.25) (layer B.Cu) (net 35))
-  (segment (start 194.2 153.25) (end 194.5 153.25) (width 0.25) (layer B.Cu) (net 35))
-  (segment (start 194.5 153.25) (end 202.5 153.25) (width 0.25) (layer B.Cu) (net 35))
-  (segment (start 202.5 153.25) (end 210.4 153.25) (width 0.25) (layer B.Cu) (net 35))
-  (segment (start 210.4 153.25) (end 214.3125 149.3375) (width 0.25) (layer B.Cu) (net 35))
-  (segment (start 194.25 153.25) (end 194.2 153.25) (width 0.25) (layer B.Cu) (net 35))
   (segment (start 233.3625 149.3375) (end 214.3125 149.3375) (width 0.25) (layer B.Cu) (net 35))
   (segment (start 339.75 147.45) (end 339.55 147.45) (width 0.25) (layer B.Cu) (net 35))
@@
   (segment (start 172.94125 140.46625) (end 176.2125 143.7375) (width 0.25) (layer B.Cu) (net 39))
   (segment (start 172.94125 140.46625) (end 169.2075 140.46625) (width 0.25) (layer B.Cu) (net 39))
-  (segment (start 188.2575 140.46625) (end 188.2575 147.3075) (width 0.25) (layer B.Cu) (net 40))
-  (segment (start 188.2575 147.3075) (end 190.75 149.8) (width 0.25) (layer B.Cu) (net 40))
+  (segment (start 188.2575 147.25) (end 188.2575 148.4425) (width 0.25) (layer B.Cu) (net 40))
+  (segment (start 188.2575 148.4425) (end 186.7 150) (width 0.25) (layer B.Cu) (net 40) (status 800000))
+  (segment (start 188.2575 140.46625) (end 188.2575 147.25) (width 0.25) (layer B.Cu) (net 40))
+  (segment (start 188.2575 147.25) (end 188.2575 147.3075) (width 0.25) (layer B.Cu) (net 40))
   (segment (start 214.3125 145.9375) (end 214.3125 143.7375) (width 0.25) (layer B.Cu) (net 41))
   (segment (start 211.04125 140.46625) (end 214.3125 143.7375) (width 0.25) (layer B.Cu) (net 41))
@@
   (segment (start 116.46625 178.56625) (end 112.0575 178.56625) (width 0.25) (layer B.Cu) (net 62))
   (segment (start 235.75 179.5) (end 236.5 178.75) (width 0.25) (layer B.Cu) (net 63))
-  (segment (start 261.05 178.75) (end 263.3 181) (width 0.25) (layer B.Cu) (net 63) (status 800000))
+  (segment (start 261.05 178.75) (end 263.3 181) (width 0.25) (layer B.Cu) (net 63))
   (segment (start 236.5 178.75) (end 261.05 178.75) (width 0.25) (layer B.Cu) (net 63))
   (segment (start 234.125 181.125) (end 235.75 179.5) (width 0.25) (layer B.Cu) (net 63))
