File: DK60TP/Kicad/DK60TP.kicad_pcb (KiCad board)
At the start: 2 copper layers, 285 x 94.5 mm, 277 parts, among them J1 USB_mini_micro_B, K1 K00, K10 K11, K11 K21, K12 K31, K13 K41, K14 K41, K15 K02, K16 K12, K17 K22, K18 K32, K19 K42, K2 K10, K20 K42, K21 K03, K22 K13, K23 K23, K24 K33, K27 K04, K28 K14, K29 K24, K3 K20, K30 K34, K32 K05, K33 K15, K34 K25, K35 K35, K38 K06, K39 K16, K4 K20, K40 K26, K41 K36, K42 K46, K44 K46, K45 K46, K46 K07, K47 K17, K48 K27, K49 K37, K5 K30, K50 K08, K51 K18, K52 K28, K53 K38, K54 K09, K55 K19, K56 K29, K57 K39, K58 K49, K59 K0A, K6 K30, K60 K1A, K61 K2A, K62 K3A, K63 K4A, K64 K4A, K65 K0B, K66 K1B, K67 K2B, K68 K3B, K69 K4B, K7 K40, K70 K4B, K71 K4B, K72 K0C, K73 K1C, K74 K2C, K75 K3C, K76 K4C, K77 K4C, K78 K0D, K79 K0D, K8 K40, K80 K1D, K81 K2D, K82 K1D, K83 K3D, K84 K3C, K85 K4D, K86 K4D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

Commit message: - Updated routing - Updated LED_TH_BIVAR
Parts:
- moved C10 9.74 mm to (216.0, 113.5), turned to 0 degrees
- moved R5 6.57 mm to (211.5, 106.5), turned to 180 degrees
- moved U1 6.01 mm to (214.5, 103.0), turned to 0 degrees
- moved C11 3.11 mm to (211.3, 109.8), turned to 0 degrees
- moved D32 2.18 mm to (172.5, 57.0)
- moved D45 1.33 mm to (228.5, 57.0)
- moved D55 1.24 mm to (265.3, 57.0)
- moved D37 1.24 mm to (191.0, 57.0)
- moved D41 1.24 mm to (210.0, 57.0)
- moved D50 1.24 mm to (247.3, 57.0)
- moved C3 0.87 mm to (133.8, 94.8), turned to 90 degrees
- moved D15 0.25 mm to (100.0, 107.0)
Connections:
- U0 pad 18: /ColA -> /ColC
- U0 pad 21: /ColC -> /ColA
Routing:
- net GND: track 246.3 -> 343.6 mm
- net /Row1: track 349.4 -> 422.6 mm
- net LED_AN: track 1714.8 -> 1784.4 mm, vias 28 -> 19
- net LED_CATH: track 1677.4 -> 1717.9 mm, vias 30 -> 18
- net Net-(D64-Pad2): track 53.3 -> 33.2 mm
- net /Col9: track 289.1 -> 272.0 mm, vias 5 -> 4
- net VCC: track 515.8 -> 529.3 mm
- net /Col0: track 194.3 -> 203.0 mm, vias 0 -> 1
- net Net-(R3-Pad1): track 132.8 -> 139.2 mm
- net /Col6: track 144.0 -> 138.8 mm
- net BACKLIT: track 88.7 -> 83.7 mm
- net /ColA: track 229.8 -> 234.6 mm, vias 3 -> 2
- net Net-(D1-Pad2): track 20.4 -> 25.1 mm
- net Net-(D35-Pad2): track 38.5 -> 34.4 mm
- net /ColC: track 285.0 -> 281.1 mm
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
Commit message: - DK60TP: Updated layout possibility - DK60TP: Split schematic in some files
Parts:
- added D146: LED, Footprint:LED_TH_BIVAR, F.Cu at (302.6, 74.1)
- added D147: LED, Footprint:LED_TH_BIVAR, F.Cu at (297.7, 93.2)
- added D148: LED, Footprint:LED_TH_BIVAR, F.Cu at (272.7, 93.2)
- added K25: K2D, Footprint:Mx_125, F.Cu at (302.4, 69.1)
- added K26: K3D, Footprint:Mx_175, F.Cu at (297.7, 88.1)
- added K31: K3C, Footprint:Mx_100, F.Cu at (271.5, 88.1)
- K82: value K1D -> K2D
- moved D136 10.2 mm to (300.0, 55.1), turned to 180 degrees
- moved D62 2.46 mm to (292.5, 95.5)
- turned K80 to 0 degrees
Connections:
- net /CAPS_LED renamed CAPS_LED
- net /Col0 renamed Col0
- net /Col1 renamed Col1
- net /Col2 renamed Col2
- net /Col3 renamed Col3
- net /Col4 renamed Col4
- net /Col5 renamed Col5
- net /Col6 renamed Col6
- net /Col7 renamed Col7
- net /Col8 renamed Col8
- net /Col9 renamed Col9
- net /ColA renamed ColA
- net /ColB renamed ColB
- net /ColC renamed ColC
- net /ColD renamed ColD
- net /Row0 renamed Row0
- net /Row1 renamed Row1
- net /Row2 renamed Row2
- net /Row3 renamed Row3
- net /Row4 renamed Row4
- K82 pad 2: Net-(D65-Pad2) -> Net-(D66-Pad2)
- U0 pad 35: Net-(U0-Pad35) -> GND
Routing:
- net Net-(D66-Pad2): track 20.0 -> 52.0 mm
- net ColD: track 339.9 -> 359.1 mm, vias 2 -> 3
- net Net-(D67-Pad2): track 12.6 -> 31.4 mm
- net Net-(D62-Pad2): track 24.4 -> 42.2 mm
- net Net-(D65-Pad2): track 37.0 -> 19.5 mm
- net GND: track 343.6 -> 355.0 mm, vias 25 -> 26
- net LED_CATH: track 1717.9 -> 1724.9 mm, vias 18 -> 19
- net Row4: track 374.6 -> 380.9 mm
- net ColC: track 281.1 -> 285.4 mm
- net VCC: track 529.3 -> 532.2 mm
- net Row0: track 416.8 -> 418.5 mm
- net Row2: track 278.4 -> 277.3 mm
- net LED_AN: track 1784.4 -> 1784.8 mm, vias 19 -> 21

Commit message: - DK60TP: Moved Matrix in separate schematic file - DK60TP: Added holes in schematic file
Parts:
- removed Poker_oval_hole (x3): VAL**, Footprint:Poker_oval_hole
- removed Poker_side_edge_long (x2): VAL**, Footprint:Poker_side_edge_long
- removed REF** (x2): MountingHole_2.2mm_M2_Pad, Mounting_Holes:MountingHole_2.2mm_M2_Pad
- added MH1: MIDDLE_LEFT, Footprint:Poker_side_edge_long, F.Cu at (29.0, 78.3)
- added MH2: TOP_LEFT, Mounting_Holes:MountingHole_2.5mm_Pad, F.Cu at (54.2, 49.8)
- added MH3: CENTER, Footprint:Poker_oval_hole, F.Cu at (157.2, 68.9)
- added MH4: BOTTOM_RIGHT, Footprint:Poker_oval_hole, F.Cu at (219.5, 107.1)
- added MH5: TOP_RIGHT, Footprint:Poker_oval_hole, F.Cu at (289.1, 49.8)
- added MH6: MIDDLE_RIGHT, Footprint:Poker_side_edge_long, F.Cu at (314.0, 78.4)
- added MH7: TRACKPOINT, Mounting_Holes:MountingHole_6mm, F.Cu at (157.2, 78.6)
Connections:
- net Net-(C1-Pad1) renamed XTAL1
- net Net-(C2-Pad1) renamed XTAL2
- net Net-(R1-Pad2) renamed RESET
- K50 pad 1: Col8 -> Net-(K50-Pad1)
- K50 pad 2: Net-(D40-Pad2) -> Net-(K50-Pad2)
- X1 pad 3: GND -> Net-(X1-Pad3)
Routing:
- net Col8: track 156.2 -> 146.7 mm
- net Net-(K50-Pad1): track 0.00 -> 9.52 mm
- net Net-(X1-Pad3): track 0.00 -> 4.23 mm
- net GND: track 355.0 -> 350.7 mm
- net LED_AN: track 1784.8 -> 1781.1 mm
- net Net-(K50-Pad2): track 0.00 -> 2.40 mm
- net Net-(D40-Pad2): track 16.5 -> 14.1 mm
- net Col6: track 138.8 -> 140.3 mm
- net Row2: track 277.3 -> 278.1 mm
- net ColD: track 359.1 -> 359.7 mm

Commit message: - DK60TP: Added RGB underglow
Parts:
- removed G*** (x2): LOGO, Footprint:darkou
- removed G***: LOGO, Footprint:OPEN-HARDWARE
- added C12: 0.1u, Capacitors_SMD:C_0805_HandSoldering, B.Cu at (53.8, 109.6)
- added C13: 0.1u, Capacitors_SMD:C_0805_HandSoldering, B.Cu at (77.8, 48.1)
- added C14: 0.1u, Capacitors_SMD:C_0805_HandSoldering, B.Cu at (172.5, 47.6)
- added C15: 0.1u, Capacitors_SMD:C_0805_HandSoldering, B.Cu at (267.3, 49.4)
- added C16: 0.1u, Capacitors_SMD:C_0805_HandSoldering, B.Cu at (290.6, 112.3)
- added D149: WS2812B, Footprint:WS2812B, B.Cu at (54.0, 104.6)
- added D150: WS2812B, Footprint:WS2812B, B.Cu at (76.3, 41.4)
- added D151: WS2812B, Footprint:WS2812B, B.Cu at (171.5, 41.9)
- added D152: WS2812B, Footprint:WS2812B, B.Cu at (267.0, 42.6)
- added D153: WS2812B, Footprint:WS2812B, B.Cu at (290.5, 106.4)
- added J2: 3PIN, Pin_Headers:Pin_Header_Straight_1x03, F.Cu at (290.5, 99.5)
- added MH10: OpenHardware, Footprint:OPEN-HARDWARE, B.Cu at (191.1, 54.7)
- added MH8: DARKOU-FRONT, Footprint:darkou, F.Cu at (131.8, 105.4)
- added MH9: DARKOU-BACK, Footprint:darkou, B.Cu at (214.2, 80.5)
- moved D63 17.6 mm to (268.8, 102.5)
- moved D58 4.47 mm to (265.2, 102.5)
- moved D5 4.18 mm to (53.5, 112.1), turned to 180 degrees
- moved U1 1.29 mm to (213.3, 103.1)
- moved D62 1.11 mm to (292.5, 94.4)
Connections:
- U0 pad 26: Net-(U0-Pad26) -> Col6
- U0 pad 27: Col6 -> RGB
Routing:
- net VCC: track 532.2 -> 927.8 mm, vias 6 -> 12
- net GND: track 350.7 -> 485.9 mm, vias 26 -> 33
- net Net-(D152-Pad2): track 0.00 -> 114.9 mm, vias 0 -> 6
- net Net-(D150-Pad2): track 0.00 -> 96.9 mm, vias 0 -> 2
- net Net-(D151-Pad2): track 0.00 -> 94.7 mm
- net RGB: track 0.00 -> 88.7 mm, vias 0 -> 2
- net Net-(D149-Pad2): track 0.00 -> 88.1 mm, vias 0 -> 4
- net LED_AN: track 1781.1 -> 1724.4 mm, vias 21 -> 28
- net LED_CATH: track 1724.9 -> 1695.6 mm, vias 19 -> 22
- net Net-(D40-Pad2): track 14.1 -> 0.00 mm
- net Col8: track 146.7 -> 133.2 mm
- net DOUT: track 0.00 -> 11.8 mm
- net Net-(K50-Pad1): track 9.52 -> 0.00 mm
- net CAPS_LED: track 106.9 -> 99.0 mm
- net Net-(D63-Pad2): track 8.22 -> 13.3 mm
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
Commit message: - DK60TP: Some changes on PCB (routing)
Parts:
- moved R1 3.00 mm to (137.5, 98.5)
- moved C13 2.61 mm to (78.0, 50.8)
- moved D150 1.87 mm to (76.5, 43.2)
- moved D67 1.52 mm to (309.2, 94.0)
- moved D151 0.85 mm to (171.5, 42.8)
Routing:
- net GND: track 485.9 -> 588.1 mm, vias 33 -> 29
- net LED_AN: track 1724.4 -> 1670.9 mm, vias 28 -> 19
- net LED_CATH: track 1695.6 -> 1646.9 mm, vias 22 -> 16
- net Net-(D152-Pad2): track 114.9 -> 88.6 mm
- net Net-(D66-Pad2): track 52.0 -> 39.2 mm
- net ColD: track 359.7 -> 367.4 mm
- net RESET: track 118.3 -> 110.9 mm
- net Net-(D149-Pad2): track 88.1 -> 80.7 mm
- net Col5: track 195.9 -> 190.0 mm
- net Net-(R3-Pad1): track 139.6 -> 135.4 mm
- net Net-(D65-Pad2): track 21.4 -> 24.5 mm
- net Net-(D67-Pad2): track 31.4 -> 28.8 mm
- net Row3: track 280.3 -> 278.5 mm, vias 2 -> 0
- net ColB: track 258.5 -> 256.8 mm
- net Net-(D7-Pad2): track 14.2 -> 13.1 mm
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
Commit message: - DK60TP: All in one PCB
Parts:
- added DM34: D, Footprint:D_SOD123, B.Cu at (148.0, 123.1)
- added DM44: D, Footprint:D_SOD123, B.Cu at (167.0, 123.1)
- added DM54: D, Footprint:D_SOD123, B.Cu at (187.7, 123.1)
- added HOLE_M2.6: VAL**, Footprint:HOLE_M2.6, F.Cu at (330.9, 119.8)
- added KM340: LMB, Footprint:Mx_100, F.Cu at (138.2, 128.7)
- added KM341: KEYSW, Footprint:Mx_125, F.Cu at (135.9, 128.7)
- added KM440: MMB, Footprint:Mx_100, F.Cu at (157.3, 128.7)
- added KM540: KEYSW, Footprint:Mx_100, F.Cu at (176.3, 128.7)
- added KM541: KEYSW, Footprint:Mx_125, F.Cu at (178.7, 128.7)
- added M1: MISC, Footprint:BreakHoles, F.Cu at (311.3, 116.4)
- added M2: MISC, Footprint:BreakHoles, F.Cu at (311.2, 119.5)
- added M3: MISC, Footprint:BreakHoles, F.Cu at (31.8, 119.5)
- added M4: MISC, Footprint:BreakHoles, F.Cu at (31.8, 116.4)
- added P1: CONN_02X04, Pin_Headers:Pin_Header_Angled_2x04, B.Cu at (203.0, 103.8)
- added P3: TRACKPOINT, Pin_Headers:Pin_Header_Angled_1x05, B.Cu at (285.3, 124.4)
- J2: moved to B.Cu
- P2: value CONN_02X05 -> MAIN_BOARD; footprint Pin_Headers:Pin_Header_Angled_2x05 -> Pin_Headers:Pin_Header_Angled_2x04
- R5: value R -> 0.5
- R7: value 100K -> 4.7K
- R9: value 4.7K -> 100K
- moved P2 123.8 mm to (83.5, 134.1), turned to 0 degrees
- moved R8 42.1 mm to (213.8, 129.2), turned to 270 degrees
- moved R9 38.9 mm to (223.3, 130.4), turned to 90 degrees
- moved R7 32.8 mm to (207.6, 129.2)
- moved C9 31.4 mm to (201.3, 127.7)
- moved J2 1.76 mm to (289.3, 98.2), turned to 90 degrees
- moved D62 1.46 mm to (292.6, 92.9)
Connections:
- P2 pad 1: Net-(P2-Pad1) -> VCC
- P2 pad 2: D5 -> GND
- P2 pad 3: Col5 -> /TRACKPOINT/Col5
- P2 pad 4: VCC -> /TRACKPOINT/D2
- P2 pad 5: Col4 -> /TRACKPOINT/Col4
- P2 pad 6: GND -> /TRACKPOINT/D5
- P2 pad 7: Col3 -> /TRACKPOINT/Col3
- P2 pad 8: Net-(C9-Pad1) -> /TRACKPOINT/Row4
- R7 pad 1: Net-(C9-Pad1) -> VCC
- R7 pad 2: GND -> /TRACKPOINT/D5
- R8 pad 2: D2 -> /TRACKPOINT/D2
- R9 pad 1: VCC -> Net-(C9-Pad1)
- R9 pad 2: D5 -> GND
Routing:
- net GND: track 588.1 -> 793.2 mm
- net /TRACKPOINT/D5: track 0.00 -> 202.8 mm, vias 0 -> 1
- net /TRACKPOINT/D2: track 0.00 -> 201.9 mm, vias 0 -> 1
- net VCC: track 928.8 -> 1121.7 mm, vias 12 -> 13
- net /TRACKPOINT/Col5: track 0.00 -> 110.9 mm
- net /TRACKPOINT/Row4: track 0.00 -> 103.8 mm
- net /TRACKPOINT/Col4: track 0.00 -> 84.0 mm
- net Net-(C9-Pad1): track 25.5 -> 85.3 mm
- net /TRACKPOINT/Col3: track 0.00 -> 55.0 mm
- net D2: track 92.5 -> 68.4 mm
- net Net-(DM34-Pad2): track 0.00 -> 10.0 mm
- net Net-(DM54-Pad2): track 0.00 -> 9.29 mm
- net Net-(DM44-Pad2): track 0.00 -> 7.59 mm
- net D5: track 74.0 -> 67.5 mm
- net Net-(D152-Pad2): track 88.6 -> 85.3 mm
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Other:
- board size 285 x 94.5 mm -> 285 x 116 mm

Commit message: - DK60TP: Added holes for Mouse button's PCB
Parts:
- added MH11: MB_LEFT, Footprint:Poker_oval_hole, F.Cu at (47.6, 131.0)
- added MH12: MB_CENTER, Footprint:Poker_oval_hole, F.Cu at (147.8, 129.2)
- added MH13: MB_RIGHT, Footprint:Poker_oval_hole, F.Cu at (304.8, 126.2)
- moved DM34 21.6 mm to (126.3, 122.9)
Routing:
- net Net-(DM34-Pad2): track 10.0 -> 14.9 mm
- net /TRACKPOINT/D5: track 202.8 -> 203.8 mm

Commit message: - DK60TP: Added RGB underglow on Mouse PCB
Parts:
- added C17: 0.1u, Capacitors_SMD:C_0805_HandSoldering, B.Cu at (55.8, 125.4)
- added C18: 0.1u, Capacitors_SMD:C_0805_HandSoldering, B.Cu at (160.8, 132.9)
- added C19: 0.1u, Capacitors_SMD:C_0805_HandSoldering, B.Cu at (291.6, 127.2)
- added D154: WS2812B, Footprint:WS2812B, B.Cu at (38.1, 127.9)
- added D155: WS2812B, Footprint:WS2812B, B.Cu at (166.8, 127.9)
- added D156: WS2812B, Footprint:WS2812B, B.Cu at (296.6, 127.9)
- J2: footprint Pin_Headers:Pin_Header_Straight_1x03 -> Pin_Headers:Pin_Header_Angled_1x03
- P1, P2: footprint Pin_Headers:Pin_Header_Angled_2x04 -> Pin_Headers:Pin_Header_Angled_2x05
- moved P2 10.6 mm to (72.8, 134.2)
- moved J2 4.32 mm to (293.6, 97.4), turned to 180 degrees
- moved D153 2.43 mm to (288.1, 106.4)
- moved DM44 1.97 mm to (168.1, 121.4), turned to 0 degrees
- moved DM34 1.52 mm to (124.8, 123.2)
- moved C16 1.29 mm to (289.3, 112.4)
Routing:
- net Net-(D154-Pad2): track 0.00 -> 135.6 mm
- net Net-(D155-Pad2): track 0.00 -> 135.2 mm
- net GND: track 793.2 -> 904.6 mm, vias 29 -> 30
- net DOUT: track 13.0 -> 117.8 mm, vias 1 -> 3
- net VCC: track 1121.7 -> 1212.2 mm, vias 13 -> 15
- net Row4: track 376.9 -> 435.8 mm, vias 2 -> 5
- net /TRACKPOINT/RGB: track 0.00 -> 38.8 mm
- net /TRACKPOINT/Col3: track 55.0 -> 72.1 mm
- net /TRACKPOINT/Col5: track 110.9 -> 124.4 mm
- net /TRACKPOINT/Col4: track 84.0 -> 97.4 mm
- net /TRACKPOINT/Row4: track 103.9 -> 115.5 mm
- net /TRACKPOINT/D2: track 201.8 -> 212.4 mm
- net /TRACKPOINT/D5: track 203.8 -> 214.4 mm
- net Net-(DM44-Pad2): track 7.59 -> 10.9 mm
- net Net-(D152-Pad2): track 85.3 -> 82.7 mm
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