File: DK60TP/Kicad/DK60TP.kicad_pcb (KiCad board)
At the start: 2 copper layers, 285 x 116 mm, 318 parts, among them J1 USB_mini_micro_B, J2 3PIN, K1 K00, K10 K11, K11 K21, K12 K31, K13 K41, K14 K41, K15 K02, K16 K12, K17 K22, K18 K32, K19 K42, K2 K10, K20 K42, K21 K03, K22 K13, K23 K23, K24 K33, K25 K2D, K26 K3D, K27 K04, K28 K14, K29 K24, K3 K20, K30 K34, K31 K3C, K32 K05, K33 K15, K34 K25, K35 K35, K38 K06, K39 K16, K4 K20, K40 K26, K41 K36, K42 K46, K44 K46, K45 K46, K46 K07, K47 K17, K48 K27, K49 K37, K5 K30, K50 K08, K51 K18, K52 K28, K53 K38, K54 K09, K55 K19, K56 K29, K57 K39, K58 K49, K59 K0A, K6 K30, K60 K1A, K61 K2A, K62 K3A, K63 K4A, K64 K4A, K65 K0B, K66 K1B, K67 K2B, K68 K3B, K69 K4B, K7 K40, K70 K4B, K71 K4B, K72 K0C, K73 K1C, K74 K2C, K75 K3C, K76 K4C, K77 K4C, K78 K0D, K79 K0D, K8 K40, K80 K1D, K81 K2D, K82 K2D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

Commit message: - DK60TP: Replaced connector for trackpoint (Molex PicoBlade)
Parts:
- P1, P2: footprint Pin_Headers:Pin_Header_Angled_2x05 -> Connectors_Molex:Molex_PicoBlade_53048-1010_10x1.25mm_Angled
- P3: footprint Pin_Headers:Pin_Header_Angled_1x05 -> Connectors_Molex:Molex_PicoBlade_53048-0510_05x1.25mm_Angled
- moved P2 11.5 mm to (69.6, 123.2), turned to 270 degrees
- moved P1 10.1 mm to (199.8, 113.4), turned to 90 degrees
- moved P3 9.75 mm to (285.1, 134.2), turned to 90 degrees
- moved R9 2.61 mm to (222.6, 132.9), turned to 270 degrees
- moved R8 2.55 mm to (214.3, 131.7)
Connections:
- P1 pad 3: Col5 -> Col3
- P1 pad 4: D2 -> Col4
- P1 pad 5: Col4 -> Col5
- P1 pad 7: Col3 -> D2
- P2 pad 3: /TRACKPOINT/Col5 -> /TRACKPOINT/Col3
- P2 pad 4: /TRACKPOINT/D2 -> /TRACKPOINT/Col4
- P2 pad 5: /TRACKPOINT/Col4 -> /TRACKPOINT/Col5
- P2 pad 7: /TRACKPOINT/Col3 -> /TRACKPOINT/D2
Routing:
- net VCC: track 1212.2 -> 1366.0 mm
- net GND: track 904.6 -> 892.7 mm, vias 30 -> 32
- net /TRACKPOINT/D2: track 212.4 -> 223.8 mm
- net /TRACKPOINT/Col4: track 97.4 -> 89.3 mm
- net /TRACKPOINT/Row4: track 115.5 -> 123.5 mm
- net /TRACKPOINT/D5: track 214.4 -> 222.4 mm
- net Row4: track 435.8 -> 443.8 mm
- net /TRACKPOINT/Col3: track 72.1 -> 65.1 mm, vias 0 -> 1
- net /TRACKPOINT/RGB: track 38.8 -> 33.8 mm, vias 0 -> 1
- net Col5: track 190.2 -> 194.8 mm
- net Col4: track 232.3 -> 235.9 mm
- net DOUT: track 117.8 -> 121.0 mm
- net Net-(C9-Pad1): track 85.3 -> 87.7 mm
- net Col3: track 257.8 -> 260.1 mm
- net /TRACKPOINT/Col5: track 124.4 -> 123.0 mm
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
Commit message: - DK60TP: Updated routing
Parts:
- J2: footprint Pin_Headers:Pin_Header_Angled_1x03 -> Connectors_Molex:Molex_PicoBlade_53048-0310_03x1.25mm_Angled
- moved C16 4.25 mm to (293.6, 112.4), turned to 0 degrees
- moved J2 3.64 mm to (292.6, 100.9), turned to 90 degrees
- moved D149 1.47 mm to (53.8, 103.2)
- moved C10 1.29 mm to (217.3, 113.4)
- moved D153 1.00 mm to (288.1, 107.4)
- moved D5 0.74 mm to (52.8, 112.4)
- moved C12 0.71 mm to (53.8, 108.9)
- moved R2 0.57 mm to (109.8, 105.7)
- moved D53 0.45 mm to (242.3, 101.7)
- moved R9 0.25 mm to (222.6, 133.2)
Routing:
- net VCC: track 1366.0 -> 1550.6 mm, vias 15 -> 16
- net GND: track 892.7 -> 870.8 mm, vias 32 -> 29
- net DOUT: track 121.0 -> 133.0 mm, vias 3 -> 0
- net /TRACKPOINT/Col5: track 123.0 -> 111.7 mm
- net /TRACKPOINT/RGB: track 33.8 -> 39.6 mm
- net /TRACKPOINT/D2: track 223.8 -> 218.7 mm
- net Row0: track 415.2 -> 420.2 mm
- net /TRACKPOINT/Col4: track 89.3 -> 93.2 mm
- net Row3: track 279.8 -> 282.7 mm
- net /TRACKPOINT/D5: track 222.4 -> 225.2 mm
- net Col0: track 206.7 -> 209.3 mm
- net LED_CATH: track 1649.1 -> 1651.6 mm
- net Row4: track 443.8 -> 445.6 mm, vias 5 -> 3
- net Net-(D149-Pad2): track 80.7 -> 79.1 mm
- net RGB: track 88.7 -> 87.2 mm
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
Commit message: - DK60TP: Replaced correctly RGB leds in mouse buttons PCB
Parts:
- KM540: value KEYSW -> RMB
- moved D154 258.5 mm to (296.6, 127.9)
- moved D156 258.5 mm to (38.1, 127.9)
- moved C17 239.2 mm to (294.8, 134.2), turned to 180 degrees
- moved C19 235.8 mm to (55.8, 125.7), turned to 90 degrees
- moved R5 9.91 mm to (201.8, 108.4), turned to 45 degrees
- moved P1 6.00 mm to (193.8, 113.4)
- moved U1 4.99 mm to (208.8, 105.4)
- moved LD1 4.08 mm to (30.8, 65.2)
- moved L1 2.17 mm to (220.8, 98.7), turned to 0 degrees
- moved C11 0.72 mm to (210.6, 109.7)
Routing:
- net /TRACKPOINT/RGB: track 39.6 -> 250.0 mm, vias 1 -> 0
- net VCC: track 1550.6 -> 1486.0 mm
- net GND: track 870.8 -> 901.5 mm, vias 29 -> 28
- net Net-(D154-Pad2): track 137.0 -> 149.1 mm
- net Row4: track 445.6 -> 439.6 mm
- net D2: track 68.1 -> 62.1 mm
- net D5: track 67.7 -> 61.7 mm
- net LED_CATH: track 1651.6 -> 1657.4 mm
- net BACKLIT: track 83.2 -> 78.5 mm
- net LED_AN: track 1667.8 -> 1663.6 mm
- net DOUT: track 133.0 -> 136.8 mm
- net Net-(LD1-Pad2): track 17.4 -> 20.6 mm
- net Net-(L1-Pad1): track 11.0 -> 14.1 mm
- net Net-(D28-Pad2): track 16.6 -> 19.2 mm
- net Net-(C9-Pad1): track 87.7 -> 86.0 mm
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
Commit message: - DK60TP: Updated Crystal position - DK60TP: Fixed labels for connectors - DK60TP: Updated routing
Parts:
- J2: value 3PIN -> RGB
- P1: value CONN_02X04 -> MOUSE_BOARD
- moved J2 94.0 mm to (198.6, 101.4), turned to 270 degrees
- moved R8 48.9 mm to (263.2, 132.6), turned to 90 degrees
- moved C9 40.1 mm to (241.2, 131.3), turned to 270 degrees
- moved R9 33.4 mm to (256.0, 131.3)
- moved R7 20.5 mm to (228.0, 130.8), turned to 135 degrees
- moved D153 4.70 mm to (290.1, 103.2)
- moved C17 4.68 mm to (299.5, 133.6), turned to 0 degrees
- moved C16 3.40 mm to (290.8, 110.4)
- moved C7 3.33 mm to (142.7, 99.1), turned to 270 degrees
- moved D56 2.29 mm to (269.2, 75.8)
- moved X1 2.21 mm to (142.5, 106.3)
- moved C1 2.20 mm to (145.2, 101.8)
- moved R5 2.14 mm to (202.6, 110.4)
- moved C19 1.51 mm to (55.2, 124.3), turned to 270 degrees
- moved C2 0.38 mm to (144.2, 111.1), turned to 225 degrees
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Routing:
- net VCC: track 1486.0 -> 1311.9 mm, vias 16 -> 12
- net GND: track 901.5 -> 816.9 mm
- net Net-(C9-Pad1): track 86.0 -> 44.1 mm
- net DOUT: track 136.8 -> 116.8 mm
- net Net-(D154-Pad2): track 149.1 -> 134.3 mm
- net LED_CATH: track 1657.4 -> 1644.0 mm, vias 16 -> 17
- net Net-(D152-Pad2): track 82.9 -> 73.3 mm, vias 6 -> 2
- net /TRACKPOINT/RGB: track 250.0 -> 241.3 mm
- net Net-(D155-Pad2): track 134.2 -> 141.7 mm
- net Row0: track 420.2 -> 415.4 mm
- net RGB: track 87.2 -> 83.0 mm
- net /TRACKPOINT/D5: track 225.2 -> 221.1 mm
- net Row4: track 439.6 -> 435.9 mm
- net Net-(D56-Pad2): track 14.6 -> 12.0 mm
- net /TRACKPOINT/Col4: track 93.2 -> 90.9 mm
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